File: pcb-default/pcb_default.kicad_pcb (KiCad board)
At the start: 2 copper layers, 10 parts, among them J1 USB2.0_C_v3, U1 AMS1117-3.3, U2 CH340C, U3 CH213K

Commit message: up
Other:
- board text added: "- ビア - 最小ホール直径: 0.3mm(JLCPCB)、0.6A - 最小ビア直径: ホール直径+0.2mm（推奨0.5mm） - 最小アニュラー幅: 0.05mm（推奨0.075mm） - 最小ビアホール間距離: 0.2mm - 配線 - 最小クリアランス: 0.15mm - 最小配線幅: 0.16mm(JLCPCB) - スルーホールアンニュラー幅: 0.18mm - ネット間パッドクリアランス: 0.1mm"
